File: pcb/dewlet/dewlet.kicad_sch (KiCad schematic)
At the start: 62 parts, among them CN1 2.1mm, IC1 ICS-43434, IC2 ICS-43434, J1 GPIO, J3 SPKR, J6 3.5mm, Q1 AOD417, U1 CAT24C256, U2 TPA3116D2DAD, U3 MIC5225-3.3, X1 3.5mm, X2 3.5mm

Commit message: Day 3
Connected amp directly to pi,  added mic files (???)
Parts:
- removed X1: 3.5mm, Adafruit MAX9744:TERMBLOCK_1X3-3.5MM, symbol Adafruit MAX9744-eagle-import:TERMBLOCK_1X3
- removed X2: 3.5mm, Adafruit MAX9744:4UCONN_19269, symbol Adafruit MAX9744-eagle-import:AUDIO_3.5MMJACK
Connections:
- net GPIO12/PWM0 is gone; now on net LEFTIN: J1.32 (Pin_32)
- net GPIO13/PWM1 is gone; now on net RIGHTIN: J1.33 (Pin_33)
- no-connect marks 39 -> 37

Commit message: Started on code!
Parts:
- added SW1: SW_Power, symbol Switch:SW_Push
- added SW2: SW_Vol_Up, symbol Switch:SW_Push
- added SW3: SW_Vol_Down, symbol Switch:SW_Push
- added SW4: SW_Assist, symbol Switch:SW_Push
- added SW5: SW_Media_Play, symbol Switch:SW_Push
Connections:
- net +3V3: now also SW1.1, SW2.1, SW3.1, SW4.1, SW5.1
- net GPIO17 renamed Vol_Up_Btn
- net Vol_Up_Btn: now also SW2.2
- net GPIO22 renamed Assist_Btn
- net Assist_Btn: now also SW4.2
- net GPIO23 renamed Media_Play_Btn
- net Media_Play_Btn: now also SW5.2
- net GPIO27 renamed Vol_Down_Btn
- net Vol_Down_Btn: now also SW3.2
- net GPIO3/SCL1 renamed Power_Btn
- net Power_Btn: now also SW1.2
- no-connect marks 37 -> 32

Commit message: Reformatted code, added media controls!
I added some controls for media, as well as a little more code organization!
Parts:
- removed R3, R4, R5: R_US, symbol Device:R_US
- added J2: SPKR, CONN_OSTTC022162_OST, symbol 2025-01-20_21-16-07:OSTTC022162
- added R3: 4.7K, Adafruit MAX9744:0805-NO, symbol Adafruit MAX9744-eagle-import:RESISTOR0805_NOOUTLINE
- C3, C4, C5, C6: value C -> 1uf
Connections:
- net L Audio Amp +: now also J3.1
- net L Audio Amp -: no longer C11.2, FB2.2 (P$2)
- net Neopixel Data: now also R3.1
- net R Audio Amp +: now also J2.1
- net at D6.4 (DIN): now also R3.2
- new net R Audio Amp -: C11.2, FB2.2 (P$2), J2.2
- no-connect marks 32 -> 31
